Commit message: Revert "Update package references"
This reverts commit 033391a139533e362bd350b5efabd9338f0d8a05.

File: iiwa_description/urdf/iiwa14.urdf.xacro (robot description, xacro)
@@ -2,7 +2,7 @@
 <robot name="iiwa14" xmlns:xacro="http://www.ros.org/wiki/xacro">
   <!-- Import Rviz colors -->
-  <xacro:include filename="$(find iiwa_description_ariac)/urdf/materials.xacro" />
+  <xacro:include filename="$(find iiwa_description)/urdf/materials.xacro" />
   <!--Import the lbr iiwa macro -->
-  <xacro:include filename="$(find iiwa_description_ariac)/urdf/iiwa14.xacro"/>
+  <xacro:include filename="$(find iiwa_description)/urdf/iiwa14.xacro"/>
   <xacro:arg name="hardware_interface" default="PositionJointInterface"/>
   <xacro:arg name="robot_name" default="iiwa"/>

File: iiwa_description/urdf/iiwa14.xacro (robot description, xacro)
@@ -2,9 +2,9 @@
 <robot xmlns:xacro="http://www.ros.org/wiki/xacro">
   <!-- Import all Gazebo-customization elements, including Gazebo colors -->
-  <xacro:include filename="$(find iiwa_description_ariac)/urdf/iiwa.gazebo.xacro" />
+  <xacro:include filename="$(find iiwa_description)/urdf/iiwa.gazebo.xacro" />
   <!-- Import Transmissions -->
-  <xacro:include filename="$(find iiwa_description_ariac)/urdf/iiwa.transmission.xacro" />
+  <xacro:include filename="$(find iiwa_description)/urdf/iiwa.transmission.xacro" />
   <!-- Include Utilities -->
-  <xacro:include filename="$(find iiwa_description_ariac)/urdf/utilities.xacro" />
+  <xacro:include filename="$(find iiwa_description)/urdf/utilities.xacro" />
   <!-- some constants -->
   <xacro:property name="safety_controller_k_pos" value="100" />
@@ -31,5 +31,5 @@
         <origin xyz="0 0 0" rpy="0 0 0"/>
         <geometry>
-          <mesh filename="package://iiwa_description_ariac/meshes/iiwa14/visual/link_0.stl"/>
+          <mesh filename="package://iiwa_description/meshes/iiwa14/visual/link_0.stl"/>
         </geometry>
         <material name="Grey"/>
@@ -38,5 +38,5 @@
         <origin xyz="0 0 0" rpy="0 0 0"/>
         <geometry>
-          <mesh filename="package://iiwa_description_ariac/meshes/iiwa14/collision/link_0.stl"/>
+          <mesh filename="package://iiwa_description/meshes/iiwa14/collision/link_0.stl"/>
         </geometry>
         <material name="Grey"/>
@@ -72,12 +72,12 @@
         <origin xyz="0 0 0" rpy="0 0 0"/>
         <geometry>
-          <mesh filename="package://iiwa_description_ariac/meshes/iiwa14/visual/link_1.stl"/>
-        </geometry>
-        <material name="Orange"/>
-      </visual>
-      <collision>
-        <origin xyz="0 0 0" rpy="0 0 0"/>
-        <geometry>
-          <mesh filename="package://iiwa_description_ariac/meshes/iiwa14/collision/link_1.stl"/>
+          <mesh filename="package://iiwa_description/meshes/iiwa14/visual/link_1.stl"/>
+        </geometry>
+        <material name="Orange"/>
+      </visual>
+      <collision>
+        <origin xyz="0 0 0" rpy="0 0 0"/>
+        <geometry>
+          <mesh filename="package://iiwa_description/meshes/iiwa14/collision/link_1.stl"/>
         </geometry>
         <material name="Orange"/>
@@ -107,12 +107,12 @@
         <origin xyz="0 0 0" rpy="0 0 0"/>
         <geometry>
-          <mesh filename="package://iiwa_description_ariac/meshes/iiwa14/visual/link_2.stl"/>
-        </geometry>
-        <material name="Orange"/>
-      </visual>
-      <collision>
-        <origin xyz="0 0 0" rpy="0 0 0"/>
-        <geometry>
-          <mesh filename="package://iiwa_description_ariac/meshes/iiwa14/collision/link_2.stl"/>
+          <mesh filename="package://iiwa_description/meshes/iiwa14/visual/link_2.stl"/>
+        </geometry>
+        <material name="Orange"/>
+      </visual>
+      <collision>
+        <origin xyz="0 0 0" rpy="0 0 0"/>
+        <geometry>
+          <mesh filename="package://iiwa_description/meshes/iiwa14/collision/link_2.stl"/>
         </geometry>
         <material name="Orange"/>
@@ -142,12 +142,12 @@
         <origin xyz="0 0 0" rpy="0 0 0"/>
         <geometry>
-          <mesh filename="package://iiwa_description_ariac/meshes/iiwa14/visual/link_3.stl"/>
-        </geometry>
-        <material name="Orange"/>
-      </visual>
-      <collision>
-        <origin xyz="0 0 0" rpy="0 0 0"/>
-        <geometry>
-          <mesh filename="package://iiwa_description_ariac/meshes/iiwa14/collision/link_3.stl"/>
+          <mesh filename="package://iiwa_description/meshes/iiwa14/visual/link_3.stl"/>
+        </geometry>
+        <material name="Orange"/>
+      </visual>
+      <collision>
+        <origin xyz="0 0 0" rpy="0 0 0"/>
+        <geometry>
+          <mesh filename="package://iiwa_description/meshes/iiwa14/collision/link_3.stl"/>
         </geometry>
         <material name="Orange"/>
@@ -177,12 +177,12 @@
         <origin xyz="0 0 0" rpy="0 0 0"/>
         <geometry>
-          <mesh filename="package://iiwa_description_ariac/meshes/iiwa14/visual/link_4.stl"/>
-        </geometry>
-        <material name="Orange"/>
-      </visual>
-      <collision>
-        <origin xyz="0 0 0" rpy="0 0 0"/>
-        <geometry>
-          <mesh filename="package://iiwa_description_ariac/meshes/iiwa14/collision/link_4.stl"/>
+          <mesh filename="package://iiwa_description/meshes/iiwa14/visual/link_4.stl"/>
+        </geometry>
+        <material name="Orange"/>
+      </visual>
+      <collision>
+        <origin xyz="0 0 0" rpy="0 0 0"/>
+        <geometry>
+          <mesh filename="package://iiwa_description/meshes/iiwa14/collision/link_4.stl"/>
         </geometry>
         <material name="Orange"/>
@@ -212,12 +212,12 @@
         <origin xyz="0 0 0" rpy="0 0 0"/>
         <geometry>
-          <mesh filename="package://iiwa_description_ariac/meshes/iiwa14/visual/link_5.stl"/>
-        </geometry>
-        <material name="Orange"/>
-      </visual>
-      <collision>
-        <origin xyz="0 0 0" rpy="0 0 0"/>
-        <geometry>
-          <mesh filename="package://iiwa_description_ariac/meshes/iiwa14/collision/link_5.stl"/>
+          <mesh filename="package://iiwa_description/meshes/iiwa14/visual/link_5.stl"/>
+        </geometry>
+        <material name="Orange"/>
+      </visual>
+      <collision>
+        <origin xyz="0 0 0" rpy="0 0 0"/>
+        <geometry>
+          <mesh filename="package://iiwa_description/meshes/iiwa14/collision/link_5.stl"/>
         </geometry>
         <material name="Orange"/>
@@ -247,12 +247,12 @@
         <origin xyz="0 0 0" rpy="0 0 0"/>
         <geometry>
-          <mesh filename="package://iiwa_description_ariac/meshes/iiwa14/visual/link_6.stl"/>
-        </geometry>
-        <material name="Orange"/>
-      </visual>
-      <collision>
-        <origin xyz="0 0 0" rpy="0 0 0"/>
-        <geometry>
-          <mesh filename="package://iiwa_description_ariac/meshes/iiwa14/collision/link_6.stl"/>
+          <mesh filename="package://iiwa_description/meshes/iiwa14/visual/link_6.stl"/>
+        </geometry>
+        <material name="Orange"/>
+      </visual>
+      <collision>
+        <origin xyz="0 0 0" rpy="0 0 0"/>
+        <geometry>
+          <mesh filename="package://iiwa_description/meshes/iiwa14/collision/link_6.stl"/>
         </geometry>
         <material name="Orange"/>
@@ -282,5 +282,5 @@
         <origin xyz="0 0 0" rpy="0 0 0"/>
         <geometry>
-          <mesh filename="package://iiwa_description_ariac/meshes/iiwa14/visual/link_7.stl"/>
+          <mesh filename="package://iiwa_description/meshes/iiwa14/visual/link_7.stl"/>
         </geometry>
         <material name="Grey"/>
@@ -289,5 +289,5 @@
         <origin xyz="0 0 0" rpy="0 0 0"/>
         <geometry>
-          <mesh filename="package://iiwa_description_ariac/meshes/iiwa14/collision/link_7.stl"/>
+          <mesh filename="package://iiwa_description/meshes/iiwa14/collision/link_7.stl"/>
         </geometry>
         <material name="Grey"/>

File: iiwa_description/urdf/iiwa7.urdf.xacro (robot description, xacro)
@@ -2,7 +2,7 @@
 <robot name="iiwa7" xmlns:xacro="http://www.ros.org/wiki/xacro">
   <!-- Import Rviz colors -->
-  <xacro:include filename="$(find iiwa_description_ariac)/urdf/materials.xacro" />
+  <xacro:include filename="$(find iiwa_description)/urdf/materials.xacro" />
   <!--Import the lbr iiwa macro -->
-  <xacro:include filename="$(find iiwa_description_ariac)/urdf/iiwa7.xacro"/>
+  <xacro:include filename="$(find iiwa_description)/urdf/iiwa7.xacro"/>
   <xacro:arg name="hardware_interface" default="PositionJointInterface"/>
   <xacro:arg name="robot_name" default="iiwa"/>

File: iiwa_description/urdf/iiwa7.xacro (robot description, xacro)
@@ -2,9 +2,9 @@
 <robot xmlns:xacro="http://www.ros.org/wiki/xacro">
   <!-- Import all Gazebo-customization elements, including Gazebo colors -->
-  <xacro:include filename="$(find iiwa_description_ariac)/urdf/iiwa.gazebo.xacro" />
+  <xacro:include filename="$(find iiwa_description)/urdf/iiwa.gazebo.xacro" />
   <!-- Import Transmissions -->
-  <xacro:include filename="$(find iiwa_description_ariac)/urdf/iiwa.transmission.xacro" />
+  <xacro:include filename="$(find iiwa_description)/urdf/iiwa.transmission.xacro" />
   <!-- Include Utilities -->
-  <xacro:include filename="$(find iiwa_description_ariac)/urdf/utilities.xacro" />
+  <xacro:include filename="$(find iiwa_description)/urdf/utilities.xacro" />
   <!-- some constants -->
   <xacro:property name="safety_controller_k_pos" value="100" />
@@ -29,12 +29,12 @@
         <origin xyz="0 0 0" rpy="0 0 0"/>
         <geometry>
-          <mesh filename="package://iiwa_description_ariac/meshes/iiwa7/visual/link_0.stl"/>
-        </geometry>
-        <material name="Grey"/>
-      </visual>
-      <collision>
-        <origin xyz="0 0 0" rpy="0 0 0"/>
-        <geometry>
-          <mesh filename="package://iiwa_description_ariac/meshes/iiwa7/collision/link_0.stl"/>
+          <mesh filename="package://iiwa_description/meshes/iiwa7/visual/link_0.stl"/>
+        </geometry>
+        <material name="Grey"/>
+      </visual>
+      <collision>
+        <origin xyz="0 0 0" rpy="0 0 0"/>
+        <geometry>
+          <mesh filename="package://iiwa_description/meshes/iiwa7/collision/link_0.stl"/>
         </geometry>
         <material name="Grey"/>
@@ -70,5 +70,5 @@
         <origin xyz="0 0 0.0075" rpy="0 0 0"/>
         <geometry>
-          <mesh filename="package://iiwa_description_ariac/meshes/iiwa7/visual/link_1.stl"/>
+          <mesh filename="package://iiwa_description/meshes/iiwa7/visual/link_1.stl"/>
         </geometry>
         <material name="Orange"/>
@@ -77,5 +77,5 @@
         <origin xyz="0 0 0.0075" rpy="0 0 0"/>
         <geometry>
-          <mesh filename="package://iiwa_description_ariac/meshes/iiwa7/collision/link_1.stl"/>
+          <mesh filename="package://iiwa_description/meshes/iiwa7/collision/link_1.stl"/>
         </geometry>
         <material name="Orange"/>
@@ -104,12 +104,12 @@
         <origin xyz="0 0 0" rpy="0 0 0"/>
         <geometry>
-          <mesh filename="package://iiwa_description_ariac/meshes/iiwa7/visual/link_2.stl"/>
-        </geometry>
-        <material name="Orange"/>
-      </visual>
-      <collision>
-        <origin xyz="0 0 0" rpy="0 0 0"/>
-        <geometry>
-          <mesh filename="package://iiwa_description_ariac/meshes/iiwa7/collision/link_2.stl"/>
+          <mesh filename="package://iiwa_description/meshes/iiwa7/visual/link_2.stl"/>
+        </geometry>
+        <material name="Orange"/>
+      </visual>
+      <collision>
+        <origin xyz="0 0 0" rpy="0 0 0"/>
+        <geometry>
+          <mesh filename="package://iiwa_description/meshes/iiwa7/collision/link_2.stl"/>
         </geometry>
         <material name="Orange"/>
@@ -138,12 +138,12 @@
         <origin xyz="0 0 -0.026" rpy="0 0 0"/>
         <geometry>
-          <mesh filename="package://iiwa_description_ariac/meshes/iiwa7/visual/link_3.stl"/>
-        </geometry>
-        <material name="Orange"/>
-      </visual>
-      <collision>
-        <origin xyz="0 0 -0.026" rpy="0 0 0"/>
-        <geometry>
-          <mesh filename="package://iiwa_description_ariac/meshes/iiwa7/collision/link_3.stl"/>
+          <mesh filename="package://iiwa_description/meshes/iiwa7/visual/link_3.stl"/>
+        </geometry>
+        <material name="Orange"/>
+      </visual>
+      <collision>
+        <origin xyz="0 0 -0.026" rpy="0 0 0"/>
+        <geometry>
+          <mesh filename="package://iiwa_description/meshes/iiwa7/collision/link_3.stl"/>
         </geometry>
         <material name="Orange"/>
@@ -172,12 +172,12 @@
         <origin xyz="0 0 0" rpy="0 0 0"/>
         <geometry>
-          <mesh filename="package://iiwa_description_ariac/meshes/iiwa7/visual/link_4.stl"/>
-        </geometry>
-        <material name="Orange"/>
-      </visual>
-      <collision>
-        <origin xyz="0 0 0" rpy="0 0 0"/>
-        <geometry>
-          <mesh filename="package://iiwa_description_ariac/meshes/iiwa7/collision/link_4.stl"/>
+          <mesh filename="package://iiwa_description/meshes/iiwa7/visual/link_4.stl"/>
+        </geometry>
+        <material name="Orange"/>
+      </visual>
+      <collision>
+        <origin xyz="0 0 0" rpy="0 0 0"/>
+        <geometry>
+          <mesh filename="package://iiwa_description/meshes/iiwa7/collision/link_4.stl"/>
         </geometry>
         <material name="Orange"/>
@@ -206,12 +206,12 @@
         <origin xyz="0 0 -0.026" rpy="0 0 0"/>
         <geometry>
-          <mesh filename="package://iiwa_description_ariac/meshes/iiwa7/visual/link_5.stl"/>
-        </geometry>
-        <material name="Orange"/>
-      </visual>
-      <collision>
-        <origin xyz="0 0 -0.026" rpy="0 0 0"/>
-        <geometry>
-          <mesh filename="package://iiwa_description_ariac/meshes/iiwa7/collision/link_5.stl"/>
+          <mesh filename="package://iiwa_description/meshes/iiwa7/visual/link_5.stl"/>
+        </geometry>
+        <material name="Orange"/>
+      </visual>
+      <collision>
+        <origin xyz="0 0 -0.026" rpy="0 0 0"/>
+        <geometry>
+          <mesh filename="package://iiwa_description/meshes/iiwa7/collision/link_5.stl"/>
         </geometry>
         <material name="Orange"/>
@@ -240,12 +240,12 @@
         <origin xyz="0 0 0" rpy="0 0 0"/>
         <geometry>
-          <mesh filename="package://iiwa_description_ariac/meshes/iiwa7/visual/link_6.stl"/>
-        </geometry>
-        <material name="Orange"/>
-      </visual>
-      <collision>
-        <origin xyz="0 0 0" rpy="0 0 0"/>
-        <geometry>
-          <mesh filename="package://iiwa_description_ariac/meshes/iiwa7/collision/link_6.stl"/>
+          <mesh filename="package://iiwa_description/meshes/iiwa7/visual/link_6.stl"/>
+        </geometry>
+        <material name="Orange"/>
+      </visual>
+      <collision>
+        <origin xyz="0 0 0" rpy="0 0 0"/>
+        <geometry>
+          <mesh filename="package://iiwa_description/meshes/iiwa7/collision/link_6.stl"/>
         </geometry>
         <material name="Orange"/>
@@ -274,5 +274,5 @@
         <origin xyz="0 0 -0.0005" rpy="0 0 0"/>
         <geometry>
-          <mesh filename="package://iiwa_description_ariac/meshes/iiwa7/visual/link_7.stl"/>
+          <mesh filename="package://iiwa_description/meshes/iiwa7/visual/link_7.stl"/>
         </geometry>
         <material name="Grey"/>
@@ -281,5 +281,5 @@
         <origin xyz="0 0 -0.0005" rpy="0 0 0"/>
         <geometry>
-          <mesh filename="package://iiwa_description_ariac/meshes/iiwa7/collision/link_7.stl"/>
+          <mesh filename="package://iiwa_description/meshes/iiwa7/collision/link_7.stl"/>
         </geometry>
         <material name="Grey"/>
